File: Project Architecture.kicad_sch (KiCad schematic)
At the start: 0 parts

Commit message: draft schematic
Other:
- removed sheet Section A - Title A
- removed sheet Section B - Title B
- added sheet ALB-MLB Toggle (toggle.kicad_sch)
- added sheet Connectors (connectors.kicad_sch)
- added sheet Motor A (motorA.kicad_sch)
- added sheet Motor Polarity Switch (motorPolarity.kicad_sch)
- added sheet MotorB (MotorB.kicad_sch)
- added sheet RotoPD (pd.kicad_sch)
- added sheet Trigger (trigger.kicad_sch)
- note removed: "Page 5"
