File: MotorB.kicad_sch (KiCad schematic)
At the start: 12 parts, among them U10 PTMUX6236RUMR, U11 TMUX7219MDGKR, U9 PINA745AIRELR

Commit message: begin pcb
Parts:
- C23: value C -> 10uF_1206_35V; footprint (none) -> Capacitor_SMD:C_0603_1608Metric_Pad1.08x0.95mm_HandSolder; symbol Device:C -> PCM_4ms_Capacitor:10uF_1206_35V; Display (none) -> 10uF; JLCPCB ID (none) -> C13585; Manufacturer (none) -> TDK; Part Number (none) -> C3216X6S1V106K160AC; Specifications (none) -> 10uF, X6S, Min 35V
- C24, C25, C28, C30: footprint (none) -> Capacitor_SMD:C_0603_1608Metric_Pad1.08x0.95mm_HandSolder; symbol Device:C_Small -> PCM_4ms_Capacitor:0.1uF_0603_16V; Display (none) -> 0.1uF; JLCPCB ID (none) -> C14663; Manufacturer (none) -> AVX Corporation; Part Number (none) -> 0603YC104KAT2A; Specifications (none) -> 0.1uF, Min. 16V 10%, X7R or X5R or similar
- C26, C27, C29, C31: footprint (none) -> Capacitor_SMD:C_0603_1608Metric_Pad1.08x0.95mm_HandSolder; symbol Device:C_Small -> PCM_4ms_Capacitor:10uF_1206_35V; Display (none) -> 10uF; JLCPCB ID (none) -> C13585; Manufacturer (none) -> TDK; Part Number (none) -> C3216X6S1V106K160AC; Specifications (none) -> 10uF, X6S, Min 35V
- U10: footprint WQFN16_RUM_TEX -> PTMUX6236RUMR:WQFN16_RUM_TEX
- U11: footprint SOIC8_DGK_TEX -> TMUX7219MDGKR:SOIC8_DGK_TEX
- U9: footprint REL0014A_PINA745AIRELR_TEX -> PINA745AIRELR:REL0014A_PINA745AIRELR_TEX
Connections:
- net +M renamed +MB
- net -M renamed -MB
