File: motorPolarity.kicad_sch (KiCad schematic)
At the start: 7 parts, among them U12 PTMUX6236RUMR

Commit message: begin pcb
Parts:
- C32, C35: footprint (none) -> Capacitor_SMD:C_0603_1608Metric_Pad1.08x0.95mm_HandSolder; symbol Device:C_Small -> PCM_4ms_Capacitor:10uF_1206_35V; Display (none) -> 10uF; JLCPCB ID (none) -> C13585; Manufacturer (none) -> TDK; Part Number (none) -> C3216X6S1V106K160AC; Specifications (none) -> 10uF, X6S, Min 35V
- C33, C34: footprint (none) -> Capacitor_SMD:C_0603_1608Metric_Pad1.08x0.95mm_HandSolder; symbol Device:C_Small -> PCM_4ms_Capacitor:0.1uF_0603_16V; Display (none) -> 0.1uF; JLCPCB ID (none) -> C14663; Manufacturer (none) -> AVX Corporation; Part Number (none) -> 0603YC104KAT2A; Specifications (none) -> 0.1uF, Min. 16V 10%, X7R or X5R or similar
- U12: footprint WQFN16_RUM_TEX -> Package_DFN_QFN:WQFN-16-1EP_4x4mm_P0.5mm_EP2.6x2.6mm_ThermalVias
