File: proalbmlb.kicad_pcb (KiCad board)
At the start: 6 copper layers, 0 parts

Commit message: begin pcb
Parts:
- added C1: 0.1μF, Capacitor_SMD:C_0603_1608Metric_Pad1.08x0.95mm_HandSolder, F.Cu at (99.0, 312.8)
- added C18: 10uF_1206_35V, Capacitor_SMD:C_0603_1608Metric_Pad1.08x0.95mm_HandSolder, F.Cu at (112.5, 312.2)
- added C19: 0.1μF, Capacitor_SMD:C_0603_1608Metric_Pad1.08x0.95mm_HandSolder, F.Cu at (119.8, 311.4)
- added C2: 10μF, Capacitor_SMD:C_0603_1608Metric_Pad1.08x0.95mm_HandSolder, F.Cu at (99.0, 311.3)
- added C20: 10μF, Capacitor_SMD:C_0603_1608Metric_Pad1.08x0.95mm_HandSolder, F.Cu at (119.8, 309.9)
- added C21: 0.1μF, Capacitor_SMD:C_0603_1608Metric_Pad1.08x0.95mm_HandSolder, F.Cu at (120.6, 319.7)
- added C22: 10μF, Capacitor_SMD:C_0603_1608Metric_Pad1.08x0.95mm_HandSolder, F.Cu at (120.6, 318.2)
- added C23: 10uF_1206_35V, Capacitor_SMD:C_0603_1608Metric_Pad1.08x0.95mm_HandSolder, F.Cu at (114.9, 325.6)
- added C24: 0.1μF, Capacitor_SMD:C_0603_1608Metric_Pad1.08x0.95mm_HandSolder, F.Cu at (126.2, 322.6)
- added C25: 0.1μF, Capacitor_SMD:C_0603_1608Metric_Pad1.08x0.95mm_HandSolder, F.Cu at (119.4, 325.5)
- added C26: 10μF, Capacitor_SMD:C_0603_1608Metric_Pad1.08x0.95mm_HandSolder, F.Cu at (127.7, 322.6)
- added C27: 10μF, Capacitor_SMD:C_0603_1608Metric_Pad1.08x0.95mm_HandSolder, F.Cu at (117.9, 325.5)
- added C28: 0.1μF, Capacitor_SMD:C_0603_1608Metric_Pad1.08x0.95mm_HandSolder, F.Cu at (125.1, 329.1)
- added C29: 10μF, Capacitor_SMD:C_0603_1608Metric_Pad1.08x0.95mm_HandSolder, F.Cu at (125.1, 330.6)
- added C3: 0.1μF, Capacitor_SMD:C_0603_1608Metric_Pad1.08x0.95mm_HandSolder, F.Cu at (102.1, 319.6)
- added C30: 0.1μF, Capacitor_SMD:C_0603_1608Metric_Pad1.08x0.95mm_HandSolder, F.Cu at (134.0, 327.8)
- added C31: 10μF, Capacitor_SMD:C_0603_1608Metric_Pad1.08x0.95mm_HandSolder, F.Cu at (132.5, 327.8)
- added C32: 10μF, Capacitor_SMD:C_0603_1608Metric_Pad1.08x0.95mm_HandSolder, F.Cu at (106.0, 310.1)
- added C33: 0.1μF, Capacitor_SMD:C_0603_1608Metric_Pad1.08x0.95mm_HandSolder, F.Cu at (106.0, 311.7)
- added C34: 0.1μF, Capacitor_SMD:C_0603_1608Metric_Pad1.08x0.95mm_HandSolder, F.Cu at (106.5, 318.5)
- added C35: 10μF, Capacitor_SMD:C_0603_1608Metric_Pad1.08x0.95mm_HandSolder, F.Cu at (106.6, 319.9)
- added C4: 10μF, Capacitor_SMD:C_0603_1608Metric_Pad1.08x0.95mm_HandSolder, F.Cu at (102.1, 318.1)
- added ENC1: Encoder_Rotary_11mm_SPST_DShaft, PCM_4ms_Encoder:ROTENC-12MM-BUT, F.Cu at (58.3, 262.0)
- added ENC2: Encoder_Rotary_11mm_SPST_DShaft, PCM_4ms_Encoder:ROTENC-12MM-BUT, F.Cu at (74.4, 262.0)
- added J1: DE9_Pins_MountingHoles, Connector_Dsub:DSUB-9_Pins_Horizontal_P2.77x2.84mm_EdgePinOffset4.94mm_Housed_MountingHolesOffset4.94mm, F.Cu at (158.6, 319.6)
- added J10: Conn_01x08_Socket, Connector_Molex:Molex_PicoBlade_53047-0810_1x08_P1.25mm_Vertical, F.Cu at (78.7, 327.2)
- added J11: Conn_01x08_Socket, Connector_Molex:Molex_PicoBlade_53047-0810_1x08_P1.25mm_Vertical, F.Cu at (39.1, 315.9)
- added J2: Conn_01x08_Socket, Connector_PinHeader_2.54mm:PinHeader_1x08_P2.54mm_Vertical, F.Cu at (72.1, 286.4)
- added J3: HPF-02-01-X-S, Connector_Samtec_HPM_THT:Samtec_HPM-02-05-x-S_Straight_1x02_Pitch5.08mm, F.Cu at (86.6, 309.4)
- added J4: Conn_01x04_Socket, Connector_Molex:Molex_PicoBlade_53047-0410_1x04_P1.25mm_Vertical, F.Cu at (108.1, 327.2)
- added J5: Conn_01x04_Socket, Connector_Molex:Molex_PicoBlade_53048-0410_1x04_P1.25mm_Horizontal, F.Cu at (39.7, 329.5)
- added J6: Conn_01x04_Socket, Connector_Molex:Molex_PicoBlade_53047-0410_1x04_P1.25mm_Vertical, F.Cu at (73.9, 338.7)
- added J7: Conn_01x04_Socket, Connector_Molex:Molex_PicoBlade_53048-0410_1x04_P1.25mm_Horizontal, F.Cu at (39.0, 343.5)
- added J8: Conn_01x02_Pin, Connector_Molex:Molex_PicoBlade_53047-0210_1x02_P1.25mm_Vertical, F.Cu at (71.4, 350.6)
- added J9: Conn_01x02_Pin, Connector_Molex:Molex_PicoBlade_53048-0210_1x02_P1.25mm_Horizontal, F.Cu at (44.6, 356.9)
- added SW1: SW_DPST, Button_Switch_THT:SW_NKK_G1xJP, F.Cu at (224.5, 258.0)
- added SW2: SW_Rotary_1x3_MP, Button_Switch_THT:A_D22022LB, F.Cu at (233.0, 278.9)
- added SW3: SW_Push_LED, Button_Switch_THT:BH16NBSBB, F.Cu at (233.2, 305.0)
- added U1: ~, Audio_Module:rotopd, F.Cu at (81.6, 296.7)
- added U10: PTMUX6236RUMR, PTMUX6236RUMR:WQFN16_RUM_TEX, F.Cu at (122.8, 324.2)
- added U11: TMUX7219MDGKR, TMUX7219MDGKR:SOIC8_DGK_TEX, F.Cu at (128.6, 327.0)
- added U12: PTMUX6236RUMR, Package_DFN_QFN:WQFN-16-1EP_4x4mm_P0.5mm_EP2.6x2.6mm_ThermalVias, F.Cu at (105.0, 315.1)
- added U2: SC1176, pictures:MODULE_SC1176, F.Cu at (127.4, 293.0)
- added U3: TMUX7201RQXR, TMUX7201RQXR:WSON8_RQX_TEX-L, F.Cu at (100.5, 315.5)
- added U7: PINA745AIRELR, PINA745AIRELR:REL0014A_PINA745AIRELR_TEX, F.Cu at (113.9, 315.1)
- added U8: PTMUX6236RUMR, PTMUX6236RUMR:WQFN16_RUM_TEX, F.Cu at (121.4, 314.8)
- added U9: PINA745AIRELR, PINA745AIRELR:REL0014A_PINA745AIRELR_TEX, F.Cu at (113.6, 322.8)
Routing:
- net /Project Architecture/Motor A/-M: track 0.00 -> 25.0 mm, vias 0 -> 1
- net /Project Architecture/Motor Polarity Switch/+M: track 0.00 -> 20.4 mm, vias 0 -> 3
- net /Project Architecture/MotorB/-MB: track 0.00 -> 17.2 mm, vias 0 -> 1
- net /Project Architecture/Connectors/-MB: track 0.00 -> 16.7 mm
- net /Project Architecture/Connectors/J1_1: track 0.00 -> 16.2 mm, vias 0 -> 2
- net /Project Architecture/Connectors/J1_2: track 0.00 -> 15.0 mm, vias 0 -> 2
- net /Project Architecture/Connectors/-M: track 0.00 -> 14.0 mm, vias 0 -> 1
- net /Project Architecture/Motor A/+M: track 0.00 -> 12.4 mm, vias 0 -> 2
- net VDD: track 0.00 -> 9.20 mm
- net /Project Architecture/Connectors/J1_3: track 0.00 -> 7.73 mm, vias 0 -> 1
- net /Project Architecture/Connectors/J1_4: track 0.00 -> 6.75 mm, vias 0 -> 1
- net GND: track 0.00 -> 6.47 mm, vias 0 -> 20
- net /Project Architecture/Connectors/J1_8: track 0.00 -> 6.43 mm, vias 0 -> 1
- net /Project Architecture/Motor Polarity Switch/-M: track 0.00 -> 6.30 mm, vias 0 -> 2
- net /Project Architecture/MotorB/+MB: track 0.00 -> 5.18 mm, vias 0 -> 1
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Other:
- board outline added: 24.4 x 35.8 mm
- copper layers 6 -> 4
