File: proalbmlb.kicad_pcb (KiCad board)
At the start: 4 copper layers, 71 x 66.1 mm, 38 parts, among them J1 DE9_Pins_MountingHoles, J10 Conn_01x08_Socket, J2 Conn_01x08_Socket, J3 HPF-02-01-X-S, J4 Conn_01x04_Socket, J6 Conn_01x04_Socket, J8 Conn_01x02_Pin, U10 PTMUX6236RUMR, U11 TMUX7219MDGKR, U12 PTMUX6236RUMR, U3 TMUX7201RQXR, U7 PINA745AIRELR, U8 PTMUX6236RUMR, U9 PINA745AIRELR

Commit message: Update cap footprint
Routing:
- added copper zone on B.Cu, net +3.3V
- added copper zone on F.Cu, net +3.3V
- added copper zone on In1.Cu, net +3.3V
- added copper zone on In2.Cu, net +3.3V

Commit message: add logo to board
Parts:
- added G***: LOGO, logo:60x12, F.Cu at (147.3, 59.9)
- added fid.A: Fiducial_1mm_Mask2mm, Fiducial:Fiducial_1mm_Mask2mm, F.Cu at (177.4, 46.9)
- added fid.B: Fiducial_1mm_Mask2mm, Fiducial:Fiducial_1mm_Mask2mm, F.Cu at (116.5, 47.0)
- added fid.C: Fiducial_1mm_Mask2mm, Fiducial:Fiducial_1mm_Mask2mm, F.Cu at (116.5, 113.2)
Routing:
- net VDD: track 0.36 -> 21.2 mm, vias 3 -> 4
- net GND: vias 82 -> 83
- removed copper zone on B.Cu, net +3.3V
- removed copper zone on F.Cu, net +3.3V
- removed copper zone on In1.Cu, net +3.3V
- removed copper zone on In2.Cu, net +3.3V
Other:
- board size 71 x 66.1 mm -> 71 x 76.3 mm
- board text added: "Engineering Sample"
