File: toggle.kicad_sch (KiCad schematic)
At the start: 1 part, among them SW1 SW_DPST

Commit message: begin pcb
Parts:
- added NT3, NT4: NetTie_2, symbol Device:NetTie_2
- SW1: footprint (none) -> Button_Switch_THT:SW_NKK_G1xJP
Connections:
- net +M: now also SW1.3, NT3.1; no longer SW1.1, SW1.2
- net -M: now also SW1.1, NT4.1; no longer SW1.3, SW1.4
- new net +MB: NT3.2, SW1.4
- new net -MB: NT4.2, SW1.2
