File: trigger.kicad_sch (KiCad schematic)
At the start: 0 parts

Commit message: begin pcb
Parts:
- added C1, C3: 0.1μF, Capacitor_SMD:C_0603_1608Metric_Pad1.08x0.95mm_HandSolder, symbol PCM_4ms_Capacitor:0.1uF_0603_16V
- added C2, C4: 10μF, Capacitor_SMD:C_0603_1608Metric_Pad1.08x0.95mm_HandSolder, symbol PCM_4ms_Capacitor:10uF_1206_35V
- added SW3: SW_Push_LED, Button_Switch_THT:BH16NBSBB, symbol Switch:SW_Push_LED
- added U3: TMUX7201RQXR, TMUX7201RQXR:WSON8_RQX_TEX-L, symbol tmux720:TMUX7201RQXR
Connections:
- new net +5V: SW3.1, SW3.2
- new net +VDC: U3.8 (D)
- new net GND: C1.1, C2.1, C3.1, C4.1, U3.3 (GND)
- new net PWM: U3.6 (SEL)
- new net VDD: C1.2, C2.2, C3.2, C4.2, U3.1 (S), U3.4 (VDD), U3.7 (VSS)
